Commit message: changed a lot of naming things, arms and grippers now move and publish joint state data

File: kinova_description/urdf/movo_arms.xacro (robot description, xacro)
@@ -29,19 +29,19 @@
     </collision>
   </link>
-	<link name="left_arm_mount">
+	<link name="left_mount">
   </link>
-  <link name="right_arm_mount">
+  <link name="right_mount">
   </link>
-	 <joint name="left_arm_attach" type="fixed">
-    <child link="left_arm_mount" />
+	 <joint name="left_attach" type="fixed">
+    <child link="left_mount" />
     <parent link="root" />
-    <origin xyz="-0.2 0 0" rpy="0 0 1.5707" />
+    <origin xyz="0 -0.2 0" rpy="0 0 1.5707" />
   </joint>
-  <joint name="right_arm_attach" type="fixed">
-    <child link="right_arm_mount" />
+  <joint name="right_attach" type="fixed">
+    <child link="right_mount" />
     <parent link="root" />
-    <origin xyz="0.2 0 0" rpy="0 0 1.5707" />
+    <origin xyz="0 0.2 0" rpy="0 0 1.5707" />
   </joint>
-  <xacro:j2s7s300  base_parent="left_arm_mount" prefix="left"/>
-	<xacro:j2s7s300  base_parent="right_arm_mount" prefix="right"/>
+  <xacro:j2s7s300  base_parent="left_mount" prefix="left"/>
+  <xacro:j2s7s300  base_parent="right_mount" prefix="right"/>
 </robot>
